File: SENSOR_BOARD_KC/SENSOR_BOARD_KC.kicad_sch (KiCad schematic)
At the start: 34 parts, among them SW2 SW_Push, SW3 SW_Push, SW4 SW_Push, SW5 SW_Push, U1 BP

Commit message: Updates
Parts:
- removed C6, C8: 0.1u, Capacitor_THT:C_Disc_D5.0mm_W2.5mm_P2.50mm, symbol Device:C
- added U2: ~, Sensor_footprints:STLINK_Connect, symbol SENSOR_SYMBOLS:ST_connec
Connections:
- net at BMP1.4 (gnd), C1.2, C11.2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: now also U2.4 (gnd)
- net at U1.3V3 (3.3V): now also U2.1 (vcc)
